File: LABSI_SM_2_BOARD/main.sch (EAGLE design)
At the start: 20 parts, among them IC1 7805TV, J1 DCJ0202, U1 ATMEGA328P-PU

Commit message: Create Fluxograma_SM.pptx
Parts:
- removed R3: 1k, resistor:R-US_0207/10
- removed R4: 2k, resistor:R-US_0207/10
- removed SV1: (no value), con-lstb:MA08-2
- removed SV2: (no value), con-lstb:MA06-2
Connections:
- removed net N$12: SV1.9
- removed net N$13: SV1.11
- removed net N$14: SV1.13
- removed net N$15: SV1.15
- removed net N$9: R3.2, SV2.9
- net GND: no longer R4.1, SV1.3, SV1.6, SV1.8, SV2.12, SV2.2, SV2.4, SV2.5, SV2.6
- net RXD: no longer SV2.10, SV2.7
- net SCL: no longer SV1.10, SV1.12, SV1.5
- net SDA: no longer SV1.14, SV1.16, SV1.7
- net TXD: no longer R3.1, R4.2, SV2.8
- net VCC: no longer SV1.1, SV1.2, SV1.4, SV2.3
Other:
- note removed: "I2C"
- note removed: "SERIAL"
