File: LABSI_SM_2_BOARD/main_SM.sch (EAGLE design)
At the start: 16 parts, among them IC1 7805TV, J1 DCJ0202, U1 ATMEGA328P-PU

Commit message: Final Commit
Parts:
- added LED3: (no value), led:LED3MM
- added R3: 330R, resistor:R-US_0207/10
- added R4: (no value), rcl:R-TRIMM3296W
Connections:
- new net N$10: R4.S, U1.PC0
- new net N$8: LED3.C, R3.1
- new net N$9: R3.2, U1.PB1
- net GND: now also LED3.A, R4.E
- net VCC: now also R4.A
Other:
- moved on the sheet: LED2, R5
Changed lines of the file:
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@@
 <part name="GND6" library="supply1" library_urn="urn:adsk.eagle:library:371" deviceset="GND" device=""/>
 <part name="FRAME1" library="frames" library_urn="urn:adsk.eagle:library:229" deviceset="DINA5_P" device=""/>
+<part name="LED3" library="led" library_urn="urn:adsk.eagle:library:259" deviceset="LED" device="3MM" package3d_urn="urn:adsk.eagle:package:15797/1"/>
+<part name="R3" library="resistor" library_urn="urn:adsk.eagle:library:348" deviceset="R-US_" device="0207/10" package3d_urn="urn:adsk.eagle:package:23491/2" value="330R"/>
+<part name="GND5" library="supply1" library_urn="urn:adsk.eagle:library:371" deviceset="GND" device=""/>
+<part name="GND7" library="supply1" library_urn="urn:adsk.eagle:library:371" deviceset="GND" device=""/>
+<part name="P+4" library="supply1" library_urn="urn:adsk.eagle:library:371" deviceset="VCC" device=""/>
+<part name="R4" library="rcl" library_urn="urn:adsk.eagle:library:334" deviceset="R-TRIMM" device="3296W" package3d_urn="urn:adsk.eagle:package:26033/1"/>
 </parts>
 <sheets>
@@
 <instance part="C3" gate="G$1" x="17.78" y="55.88" smashed="yes" rot="R90">
 <attribute name="NAME" x="17.399" y="57.404" size="1.778" layer="95" rot="R90"/>
-<attribute name="VALUE" x="22.479" y="62.484" size="1.778" layer="96" rot="R180"/>
+<attribute name="VALUE" x="19.939" y="59.944" size="1.778" layer="96" rot="R270"/>
 </instance>
 <instance part="C4" gate="G$1" x="17.78" y="50.8" smashed="yes" rot="R90">
 <attribute name="NAME" x="17.399" y="47.244" size="1.778" layer="95" rot="R90"/>
-<attribute name="VALUE" x="17.399" y="44.704" size="1.778" layer="96"/>
+<attribute name="VALUE" x="22.479" y="47.244" size="1.778" layer="96" rot="R90"/>
 </instance>
 <instance part="GND4" gate="1" x="12.7" y="48.26" smashed="yes">
@@
 <attribute name="VALUE" x="12.7" y="151.13" size="1.778" layer="96"/>
 </instance>
-<instance part="LED2" gate="G$1" x="101.6" y="66.04" smashed="yes" rot="R270">
-<attribute name="NAME" x="97.028" y="62.484" size="1.778" layer="95"/>
-<attribute name="VALUE" x="97.028" y="60.325" size="1.778" layer="96"/>
-</instance>
-<instance part="R5" gate="G$1" x="86.36" y="66.04" smashed="yes" rot="R180">
-<attribute name="NAME" x="90.17" y="64.5414" size="1.778" layer="95" rot="R180"/>
-<attribute name="VALUE" x="90.17" y="69.342" size="1.778" layer="96" rot="R180"/>
-</instance>
-<instance part="GND6" gate="1" x="109.22" y="66.04" smashed="yes" rot="R90">
-<attribute name="VALUE" x="111.76" y="63.5" size="1.778" layer="96" rot="R90"/>
+<instance part="LED2" gate="G$1" x="93.98" y="83.82" smashed="yes">
+<attribute name="NAME" x="97.536" y="79.248" size="1.778" layer="95" rot="R90"/>
+<attribute name="VALUE" x="99.695" y="79.248" size="1.778" layer="96" rot="R90"/>
+</instance>
+<instance part="R5" gate="G$1" x="93.98" y="71.12" smashed="yes" rot="R270">
+<attribute name="NAME" x="95.4786" y="74.93" size="1.778" layer="95" rot="R270"/>
+<attribute name="VALUE" x="90.678" y="74.93" size="1.778" layer="96" rot="R270"/>
+</instance>
+<instance part="GND6" gate="1" x="93.98" y="91.44" smashed="yes" rot="R180">
+<attribute name="VALUE" x="96.52" y="93.98" size="1.778" layer="96" rot="R180"/>
 </instance>
 <instance part="FRAME1" gate="G$1" x="0" y="-2.54" smashed="yes">
@@
 <attribute name="LAST_DATE_TIME" x="87.63" y="7.747" size="2.286" layer="94"/>
 <attribute name="SHEET" x="100.965" y="2.667" size="2.54" layer="94"/>
+</instance>
+<instance part="LED3" gate="G$1" x="15.24" y="68.58" smashed="yes" rot="R90">
+<attribute name="NAME" x="19.812" y="72.136" size="1.778" layer="95" rot="R180"/>
+<attribute name="VALUE" x="19.812" y="74.295" size="1.778" layer="96" rot="R180"/>
+</instance>
+<instance part="R3" gate="G$1" x="27.94" y="68.58" smashed="yes">
+<attribute name="NAME" x="24.13" y="70.0786" size="1.778" layer="95"/>
+<attribute name="VALUE" x="24.13" y="65.278" size="1.778" layer="96"/>
+</instance>
+<instance part="GND5" gate="1" x="10.16" y="68.58" smashed="yes" rot="R270">
+<attribute name="VALUE" x="7.62" y="71.12" size="1.778" layer="96" rot="R270"/>
+</instance>
+<instance part="GND7" gate="1" x="111.76" y="50.8" smashed="yes">
+<attribute name="VALUE" x="109.22" y="48.26" size="1.778" layer="96"/>
+</instance>
+<instance part="P+4" gate="VCC" x="111.76" y="71.12" smashed="yes">
+<attribute name="VALUE" x="109.22" y="68.58" size="1.778" layer="96" rot="R90"/>
+</instance>
+<instance part="R4" gate="G$1" x="111.76" y="60.96" smashed="yes" rot="R180">
+<attribute name="NAME" x="117.729" y="64.77" size="1.778" layer="95" rot="R270"/>
+<attribute name="VALUE" x="115.57" y="64.77" size="1.778" layer="96" rot="R270"/>
 </instance>
 </instances>
@@
 <pinref part="LED2" gate="G$1" pin="A"/>
 <pinref part="GND6" gate="1" pin="GND"/>
-<wire x1="104.14" y1="66.04" x2="106.68" y2="66.04" width="0.1524" layer="91"/>
+<wire x1="93.98" y1="86.36" x2="93.98" y2="88.9" width="0.1524" layer="91"/>
+</segment>
+<segment>
+<pinref part="LED3" gate="G$1" pin="A"/>
+<pinref part="GND5" gate="1" pin="GND"/>
+</segment>
+<segment>
+<pinref part="GND7" gate="1" pin="GND"/>
+<pinref part="R4" gate="G$1" pin="E"/>
+<wire x1="111.76" y1="53.34" x2="111.76" y2="55.88" width="0.1524" layer="91"/>
 </segment>
 </net>
@@
 <label x="15.24" y="101.6" size="1.778" layer="95"/>
 </segment>
+<segment>
+<pinref part="P+4" gate="VCC" pin="VCC"/>
+<pinref part="R4" gate="G$1" pin="A"/>
+<wire x1="111.76" y1="68.58" x2="111.76" y2="66.04" width="0.1524" layer="91"/>
+</segment>
 </net>
 <net name="N$2" class="0">
@@
 <pinref part="R5" gate="G$1" pin="1"/>
 <pinref part="LED2" gate="G$1" pin="C"/>
-<wire x1="96.52" y1="66.04" x2="91.44" y2="66.04" width="0.1524" layer="91"/>
+<wire x1="93.98" y1="78.74" x2="93.98" y2="76.2" width="0.1524" layer="91"/>
 </segment>
 </net>
@@
 <pinref part="U1" gate="A" pin="PD6"/>
 <pinref part="R5" gate="G$1" pin="2"/>
-<wire x1="81.28" y1="66.04" x2="76.2" y2="66.04" width="0.1524" layer="91"/>
-</segment>
-</net>
+<wire x1="93.98" y1="66.04" x2="76.2" y2="66.04" width="0.1524" layer="91"/>
+</segment>
+</net>
+<net name="N$8" class="0">
+<segment>
+<pinref part="R3" gate="G$1" pin="1"/>
+<pinref part="LED3" gate="G$1" pin="C"/>
+<wire x1="20.32" y1="68.58" x2="22.86" y2="68.58" width="0.1524" layer="91"/>
+</segment>
+</net>
+<net name="N$10" class="0">
+<segment>
+<pinref part="U1" gate="A" pin="PC0"/>
+<wire x1="76.2" y1="58.42" x2="96.52" y2="58.42" width="0.1524" layer="91"/>
+<wire x1="96.52" y1="58.42" x2="96.52" y2="60.96" width="0.1524" layer="91"/>
+<wire x1="96.52" y1="60.96" x2="106.68" y2="60.96" width="0.1524" layer="91"/>
+<pinref part="R4" gate="G$1" pin="S"/>
+</segment>
+</net>
+<net name="N$9" class="0">
+<segment>
+<pinref part="U1" gate="A" pin="PB1"/>
+<wire x1="40.64" y1="66.04" x2="35.56" y2="66.04" width="0.1524" layer="91"/>
+<pinref part="R3" gate="G$1" pin="2"/>
+<wire x1="33.02" y1="68.58" x2="35.56" y2="68.58" width="0.1524" layer="91"/>
+<wire x1="35.56" y1="68.58" x2="35.56" y2="66.04" width="0.1524" layer="91"/>
+</segment>
+</net>
